File: RP2040.kicad_sch (KiCad schematic)
At the start: 32 parts, among them J1 USB_B_Micro, J2 Conn_01x12, J3 Conn_01x12, SW1 USB_BOOT, SW2 RESET, U1 AP1117-33, U2 W25Q128JVS, U3 RP2040, Y1 12MHz

Commit message: fix: Fix crystal orientation
Connections:
- net GND: now also Y1.2, Y1.4; no longer Y1.1, Y1.3
- net at C11.1, U3.20 (XIN): now also Y1.3; no longer Y1.2
- net at C13.1, U3.21 (XOUT): now also Y1.1; no longer Y1.4
Other:
- moved on the sheet: Y1
Changed lines of the file:
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@@
 	)
 	(junction
-		(at 96.52 104.14)
+		(at 134.62 85.09)
 		(diameter 0)
 		(color 0 0 0 0)
 	)
 	(junction
-		(at 134.62 95.25)
+		(at 96.52 104.14)
 		(diameter 0)
 		(color 0 0 0 0)
@@
 	)
 	(junction
-		(at 134.62 85.09)
+		(at 134.62 95.25)
 		(diameter 0)
 		(color 0 0 0 0)
@@
 	(wire
 		(pts
-			(xy 134.62 85.09) (xy 149.86 85.09)
-		)
-		(stroke
-			(width 0)
-			(type default)
-		)
-	)
-	(wire
-		(pts
 			(xy 36.83 114.3) (xy 36.83 116.84)
 		)
@@
 	(wire
 		(pts
-			(xy 111.76 104.14) (xy 111.76 106.68)
+			(xy 134.62 93.98) (xy 134.62 95.25)
 		)
 		(stroke
@@
 	(wire
 		(pts
-			(xy 31.75 30.48) (xy 33.02 30.48)
+			(xy 111.76 104.14) (xy 111.76 106.68)
 		)
 		(stroke
@@
 	(wire
 		(pts
-			(xy 33.02 39.37) (xy 41.91 39.37)
+			(xy 31.75 30.48) (xy 33.02 30.48)
 		)
 		(stroke
@@
 	(wire
 		(pts
-			(xy 138.43 90.17) (xy 139.7 90.17)
+			(xy 33.02 39.37) (xy 41.91 39.37)
 		)
 		(stroke
@@
 	(wire
 		(pts
+			(xy 134.62 85.09) (xy 134.62 86.36)
+		)
+		(stroke
+			(width 0)
+			(type default)
+		)
+	)
+	(wire
+		(pts
 			(xy 33.02 30.48) (xy 34.29 30.48)
 		)
@@
 	(wire
 		(pts
-			(xy 120.65 85.09) (xy 134.62 85.09)
+			(xy 129.54 90.17) (xy 129.54 91.44)
 		)
 		(stroke
@@
 	(wire
 		(pts
-			(xy 139.7 90.17) (xy 139.7 91.44)
+			(xy 120.65 85.09) (xy 134.62 85.09)
 		)
 		(stroke
@@
 	(wire
 		(pts
-			(xy 129.54 91.44) (xy 129.54 90.17)
-		)
-		(stroke
-			(width 0)
-			(type default)
-		)
-	)
-	(wire
-		(pts
 			(xy 55.88 62.23) (xy 90.17 62.23)
 		)
@@
 	(wire
 		(pts
-			(xy 60.96 45.72) (xy 58.42 45.72)
+			(xy 134.62 85.09) (xy 149.86 85.09)
 		)
 		(stroke
@@
 	(wire
 		(pts
-			(xy 127 138.43) (xy 127 137.16)
+			(xy 60.96 45.72) (xy 58.42 45.72)
 		)
 		(stroke
@@
 	(wire
 		(pts
-			(xy 257.81 113.03) (xy 256.54 113.03)
+			(xy 127 138.43) (xy 127 137.16)
 		)
 		(stroke
@@
 	(wire
 		(pts
-			(xy 129.54 90.17) (xy 130.81 90.17)
+			(xy 257.81 113.03) (xy 256.54 113.03)
 		)
 		(stroke
@@
 	(wire
 		(pts
+			(xy 139.7 90.17) (xy 139.7 91.44)
+		)
+		(stroke
+			(width 0)
+			(type default)
+		)
+	)
+	(wire
+		(pts
 			(xy 177.8 31.75) (xy 180.34 31.75)
 		)
@@
 	(symbol
 		(lib_id "Device:Crystal_GND24")
-		(at 134.62 90.17 0)
+		(at 134.62 90.17 90)
 		(unit 1)
 		(body_style 1)
@@
 		(fields_autoplaced yes)
 		(property "Reference" "Y1"
-			(at 142.24 85.9791 0)
+			(at 143.51 85.2168 90)
 			(show_name no)
 			(do_not_autoplace no)
@@
 		)
 		(property "Value" "12MHz"
-			(at 142.24 88.5191 0)
+			(at 143.51 87.7568 90)
 			(show_name no)
 			(do_not_autoplace no)
